File: HARDWARE/MINI-SUMO GOKU/minisumogokufinalizado 23 de septiembre.kicad_pcb (KiCad board)
At the start: 2 copper layers, 74.7 x 54 mm, 17 parts, among them J1 batterly, J2 hc-sr05, J3 sensor, M1 Motor_DC, M2 Motor_DC, SW1 SW_DPST_x2, U1 L293D, U2 L7805

Commit message: Add files via upload
Parts:
- moved C6 1.92 mm to (144.6, 112.5)
Routing:
- net +5V: track 166.8 -> 163.2 mm
